Commit message: Autonomous navigation is possible, but planning is very slow.

File: turtlebot_description/urdf/sensors/d455.urdf.xacro (robot description, xacro)
@@ -6,5 +6,5 @@
   <xacro:property name="pole_px" value="0.103" />
   <xacro:property name="pole_py" value="-0.098"/>
-  <xacro:property name="pole_pz" value="0.195" />
+  <xacro:property name="pole_pz" value="0.150" />
   <xacro:property name="d455_bracket_end_offset_py" value="0.02" />
   <xacro:property name="d455_bracket_end_offset_pz" value="0" />
